File: pcb/amp.kicad_sch (KiCad schematic)
At the start: 16 parts, among them U3 OPA2333xxD

Commit message: Update PCB
Parts:
- C10, C11, C16, C8, C9: footprint (none) -> Capacitor_SMD:C_0603_1608Metric
- R10, R11: value 1k -> 1k±0.1%; footprint (none) -> Resistor_SMD:R_0603_1608Metric
- R12, R13: value 100k -> 100k±0.1%; footprint (none) -> Resistor_SMD:R_0603_1608Metric
- R14, R23, R7: footprint (none) -> Resistor_SMD:R_0603_1608Metric
- R8, R9: value 100 -> 100±0.1%; footprint (none) -> Resistor_SMD:R_0603_1608Metric
- TP1: footprint (none) -> TestPoint:TestPoint_Pad_D1.5mm
- U3: footprint (none) -> Package_SO:SOIC-8_3.9x4.9mm_P1.27mm
Changed lines of the file:
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@@
 			)
 		)
-		(property "Value" "1k"
+		(property "Value" "1k±0.1%"
 			(at 144.78 76.2 90)
 			(show_name no)
@@
 			)
 		)
-		(property "Footprint" ""
+		(property "Footprint" "Resistor_SMD:R_0603_1608Metric"
 			(at 144.78 77.978 90)
 			(hide yes)
@@
 			)
 		)
-		(property "Value" "100k"
+		(property "Value" "100k±0.1%"
 			(at 161.29 96.5199 0)
 			(show_name no)
@@
 			)
 		)
-		(property "Footprint" ""
+		(property "Footprint" "Resistor_SMD:R_0603_1608Metric"
 			(at 156.972 95.25 90)
 			(hide yes)
@@
 			)
 		)
-		(property "Value" "100"
+		(property "Value" "100±0.1%"
 			(at 128.27 87.63 90)
 			(show_name no)
@@
 			)
 		)
-		(property "Footprint" ""
+		(property "Footprint" "Resistor_SMD:R_0603_1608Metric"
 			(at 128.27 89.408 90)
 			(hide yes)
@@
 			)
 		)
-		(property "Footprint" ""
+		(property "Footprint" "Capacitor_SMD:C_0603_1608Metric"
 			(at 115.2652 97.79 0)
 			(hide yes)
@@
 			)
 		)
-		(property "Footprint" ""
+		(property "Footprint" "TestPoint:TestPoint_Pad_D1.5mm"
 			(at 210.82 72.39 0)
 			(hide yes)
@@
 			)
 		)
-		(property "Value" "100"
+		(property "Value" "100±0.1%"
 			(at 128.27 76.2 90)
 			(show_name no)
@@
 			)
 		)
-		(property "Footprint" ""
+		(property "Footprint" "Resistor_SMD:R_0603_1608Metric"
 			(at 128.27 77.978 90)
 			(hide yes)
@@
 			)
 		)
-		(property "Footprint" ""
+		(property "Footprint" "Capacitor_SMD:C_0603_1608Metric"
 			(at 136.8552 85.09 0)
 			(hide yes)
@@
 			)
 		)
-		(property "Footprint" ""
+		(property "Footprint" "Capacitor_SMD:C_0603_1608Metric"
 			(at 159.7152 138.43 0)
 			(hide yes)
@@
 			)
 		)
-		(property "Footprint" ""
+		(property "Footprint" "Capacitor_SMD:C_0603_1608Metric"
 			(at 196.5452 91.44 0)
 			(hide yes)
@@
 			)
 		)
-		(property "Footprint" ""
+		(property "Footprint" "Resistor_SMD:R_0603_1608Metric"
 			(at 92.202 66.04 90)
 			(hide yes)
@@
 			)
 		)
-		(property "Footprint" ""
+		(property "Footprint" "Resistor_SMD:R_0603_1608Metric"
 			(at 87.122 96.52 90)
 			(hide yes)
@@
 			)
 		)
-		(property "Value" "1k"
+		(property "Value" "1k±0.1%"
 			(at 144.78 87.63 90)
 			(show_name no)
@@
 			)
 		)
-		(property "Footprint" ""
+		(property "Footprint" "Resistor_SMD:R_0603_1608Metric"
 			(at 144.78 89.408 90)
 			(hide yes)
@@
 			)
 		)
-		(property "Footprint" ""
+		(property "Footprint" "Resistor_SMD:R_0603_1608Metric"
 			(at 190.5 80.518 90)
 			(hide yes)
@@
 			)
 		)
-		(property "Footprint" ""
+		(property "Footprint" "Capacitor_SMD:C_0603_1608Metric"
 			(at 121.6152 97.79 0)
 			(hide yes)
@@
 			)
 		)
-		(property "Value" "100k"
+		(property "Value" "100k±0.1%"
 			(at 172.72 64.77 90)
 			(show_name no)
@@
 			)
 		)
-		(property "Footprint" ""
+		(property "Footprint" "Resistor_SMD:R_0603_1608Metric"
 			(at 172.72 66.548 90)
 			(hide yes)
@@
 			)
 		)
-		(property "Footprint" ""
+		(property "Footprint" "Package_SO:SOIC-8_3.9x4.9mm_P1.27mm"
 			(at 173.99 78.74 0)
 			(hide yes)

Commit message: update value
Parts:
- R10, R11: value 1k±0.1% -> 270±0.1%
Changed lines of the file:
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@@
 			)
 		)
-		(property "Value" "1k±0.1%"
+		(property "Value" "270±0.1%"
 			(at 144.78 76.2 90)
 			(show_name no)
@@
 			)
 		)
-		(property "Value" "1k±0.1%"
+		(property "Value" "270±0.1%"
 			(at 144.78 87.63 90)
 			(show_name no)
